File: Keypad PCB.kicad_pcb (KiCad board)
At the start: 2 copper layers, 20 parts, among them SW1 SW_Push, U1 ATmega32U4-AU, Y1 Crystal_GND24_Small

Commit message: Avancement sur le rooting du pcb
Parts:
- removed USB1: Molex-0548190589, random-keyboard-parts:Molex-0548190589
- added J1: Conn_01x04_Female, Connectors_JST:JST_SH_SM04B-SRSS-TB_04x1.00mm_Angled, B.Cu at (237.3, 84.1)
- SW1: moved to F.Cu
- moved C1 220.4 mm to (251.6, 112.7), turned to 0 degrees
- moved C6 218.2 mm to (247.7, 118.3), turned to 135 degrees
- moved F1 216.8 mm to (240.5, 90.5), turned to 90 degrees
- moved R2 216.3 mm to (238.1, 90.5)
- moved Y1 212.6 mm to (245.3, 120.7), turned to 45 degrees
- moved C7 212.3 mm to (243.7, 106.4), turned to 135 degrees
- moved R1 210.5 mm to (235.7, 90.5)
- moved C5 207.9 mm to (242.9, 123.0), turned to 315 degrees
- moved C2 201.5 mm to (251.6, 110.3), turned to 0 degrees
- moved C3 200.6 mm to (251.6, 108.0), turned to 0 degrees
- moved U1 197.4 mm to (237.7, 112.7), turned to 225 degrees
- moved SW1 196.6 mm to (221.5, 108.0), turned to 270 degrees
- moved R3 196.4 mm to (225.3, 107.2)
- moved C4 191.6 mm to (234.3, 103.3), turned to 225 degrees
- moved R4 181.5 mm to (230.3, 116.8), turned to 315 degrees
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Connections:
- R1 pad 2: D- -> Net-(J1-Pad2)
- R2 pad 2: D+ -> Net-(J1-Pad3)
Routing:
- net +5V: track 0.00 -> 81.3 mm
- net GND: track 0.00 -> 46.3 mm
- net Net-(R1-Pad1): track 0.00 -> 17.9 mm
- net Net-(R2-Pad1): track 0.00 -> 17.7 mm
- net Net-(C6-Pad1): track 0.00 -> 10.3 mm
- net Net-(C5-Pad1): track 0.00 -> 7.26 mm
- net Net-(R4-Pad2): track 0.00 -> 4.10 mm
- net Net-(J1-Pad2): track 0.00 -> 3.93 mm
- net VCC: track 0.00 -> 3.71 mm
- net Net-(J1-Pad3): track 0.00 -> 3.60 mm
- net Net-(C7-Pad1): track 0.00 -> 3.26 mm
Other:
- board outline added: 47 x 47 mm
- net class Power added: clearance 0.2, trace_width 0.381, via_dia 0.8, via_drill 0.4

Commit message: ça avance
Routing:
- net +5V: track 81.3 -> 0.00 mm
- net GND: track 46.3 -> 43.8 mm
- net Net-(C6-Pad1): track 10.3 -> 11.0 mm
Changed lines of the file:
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@@
     (thickness 1.6)
     (drawings 4)
-    (tracks 83)
+    (tracks 61)
     (zones 0)
     (modules 20)
@@
   (gr_line (start 215 127) (end 262 127) (layer Edge.Cuts) (width 0.05))
   (gr_line (start 215 80) (end 215 127) (layer Edge.Cuts) (width 0.05))
-  (segment (start 252.55625 107.95) (end 252.55625 114.15625) (width 0.381) (layer B.Cu) (net 1))
-  (segment (start 252.55625 114.15625) (end 252.4125 114.3) (width 0.381) (layer B.Cu) (net 1))
-  (segment (start 252.4125 114.3) (end 246.85625 114.3) (width 0.381) (layer B.Cu) (net 1))
-  (segment (start 243.50692 116.212678) (end 242.90588 115.611638) (width 0.381) (layer B.Cu) (net 1))
-  (segment (start 243.661009 116.366767) (end 243.50692 116.212678) (width 0.381) (layer B.Cu) (net 1))
-  (segment (start 244.789483 116.366767) (end 243.661009 116.366767) (width 0.381) (layer B.Cu) (net 1))
-  (segment (start 246.85625 114.3) (end 244.789483 116.366767) (width 0.381) (layer B.Cu) (net 1))
   (segment (start 244.116097 123.128479) (end 243.550413 123.694163) (width 0.381) (layer B.Cu) (net 1))
   (segment (start 245.199641 122.044935) (end 244.116097 123.128479) (width 0.381) (layer B.Cu) (net 1))
@@
   (segment (start 242.695086 124.54949) (end 239.64324 124.54949) (width 0.381) (layer B.Cu) (net 1))
   (segment (start 243.550413 123.694163) (end 242.695086 124.54949) (width 0.381) (layer B.Cu) (net 1))
-  (segment (start 243.018337 106.306792) (end 241.208823 108.116306) (width 0.381) (layer B.Cu) (net 1))
-  (segment (start 243.018337 105.699587) (end 243.018337 106.306792) (width 0.381) (layer B.Cu) (net 1))
   (segment (start 230.84971 110.343693) (end 231.45075 110.944733) (width 0.381) (layer B.Cu) (net 1))
   (segment (start 230.438863 110.343693) (end 230.84971 110.343693) (width 0.381) (layer B.Cu) (net 1))
@@
   (segment (start 229.655424 116.149174) (end 229.655424 111.127132) (width 0.381) (layer B.Cu) (net 1))
   (segment (start 235.802113 120.708363) (end 235.802113 120.311241) (width 0.381) (layer B.Cu) (net 1))
-  (segment (start 250.68125 107.95) (end 250.68125 113.3625) (width 0.381) (layer B.Cu) (net 2))
-  (segment (start 250.68125 113.3625) (end 250.5375 113.50625) (width 0.381) (layer B.Cu) (net 2))
-  (segment (start 244.072605 115.646992) (end 243.471565 115.045952) (width 0.381) (layer B.Cu) (net 2))
-  (segment (start 244.211371 115.785758) (end 244.072605 115.646992) (width 0.381) (layer B.Cu) (net 2))
-  (segment (start 244.344685 115.785758) (end 244.211371 115.785758) (width 0.381) (layer B.Cu) (net 2))
-  (segment (start 246.624193 113.50625) (end 244.344685 115.785758) (width 0.381) (layer B.Cu) (net 2))
-  (segment (start 250.5375 113.50625) (end 246.624193 113.50625) (width 0.381) (layer B.Cu) (net 2))
-  (segment (start 242.941234 108.646637) (end 242.340194 109.247677) (width 0.381) (layer B.Cu) (net 2))
-  (segment (start 243.964635 108.646637) (end 242.941234 108.646637) (width 0.381) (layer B.Cu) (net 2))
-  (segment (start 245.473398 107.137874) (end 243.964635 108.646637) (width 0.381) (layer B.Cu) (net 2))
-  (segment (start 245.473398 106.612432) (end 245.473398 107.137874) (width 0.381) (layer B.Cu) (net 2))
-  (segment (start 239.7125 100.851534) (end 245.473398 106.612432) (width 0.381) (layer B.Cu) (net 2))
-  (segment (start 239.7125 92.68125) (end 239.7125 100.851534) (width 0.381) (layer B.Cu) (net 2))
-  (segment (start 240.50625 91.8875) (end 239.7125 92.68125) (width 0.381) (layer B.Cu) (net 2))
-  (segment (start 246.285524 107.95) (end 245.473398 107.137874) (width 0.381) (layer B.Cu) (net 2))
-  (segment (start 249.53426 106.85949) (end 248.44375 107.95) (width 0.381) (layer B.Cu) (net 2))
-  (segment (start 253.06272 106.85949) (end 249.53426 106.85949) (width 0.381) (layer B.Cu) (net 2))
-  (segment (start 253.43426 107.23103) (end 253.06272 106.85949) (width 0.381) (layer B.Cu) (net 2))
-  (segment (start 253.43426 115.087365) (end 253.43426 107.23103) (width 0.381) (layer B.Cu) (net 2))
-  (segment (start 239.402578 125.1305) (end 243.391125 125.1305) (width 0.381) (layer B.Cu) (net 2))
-  (segment (start 243.391125 125.1305) (end 253.43426 115.087365) (width 0.381) (layer B.Cu) (net 2))
-  (segment (start 235.221104 119.760879) (end 235.221104 120.949026) (width 0.381) (layer B.Cu) (net 2))
-  (segment (start 235.976233 119.00575) (end 235.221104 119.760879) (width 0.381) (layer B.Cu) (net 2))
-  (segment (start 235.221104 120.949026) (end 239.402578 125.1305) (width 0.381) (layer B.Cu) (net 2))
-  (segment (start 248.44375 107.95) (end 246.285524 107.95) (width 0.381) (layer B.Cu) (net 2))
-  (segment (start 250.68125 107.95) (end 248.44375 107.95) (width 0.381) (layer B.Cu) (net 2))
+  (segment (start 243.018337 106.306792) (end 241.208823 108.116306) (width 0.381) (layer B.Cu) (net 1))
+  (segment (start 243.018337 105.699587) (end 243.018337 106.306792) (width 0.381) (layer B.Cu) (net 1))
+  (segment (start 242.30484 115.010598) (end 242.90588 115.611638) (width 0.381) (layer B.Cu) (net 1))
+  (segment (start 240.50625 113.212008) (end 242.30484 115.010598) (width 0.381) (layer B.Cu) (net 1))
+  (segment (start 241.208823 108.116306) (end 240.50625 108.818879) (width 0.381) (layer B.Cu) (net 1))
+  (segment (start 237.98904 107.02029) (end 240.50625 109.5375) (width 0.381) (layer B.Cu) (net 1))
+  (segment (start 236.577273 107.02029) (end 237.98904 107.02029) (width 0.381) (layer B.Cu) (net 1))
+  (segment (start 235.976233 106.41925) (end 236.577273 107.02029) (width 0.381) (layer B.Cu) (net 1))
+  (segment (start 240.50625 108.818879) (end 240.50625 109.5375) (width 0.381) (layer B.Cu) (net 1))
+  (segment (start 240.50625 109.5375) (end 240.50625 113.212008) (width 0.381) (layer B.Cu) (net 1))
   (segment (start 242.348332 122.368337) (end 243.889892 120.826777) (width 0.25) (layer B.Cu) (net 3))
   (segment (start 242.224587 122.368337) (end 242.348332 122.368337) (width 0.25) (layer B.Cu) (net 3))
@@
   (segment (start 243.889892 120.826777) (end 243.889892 118.858392) (width 0.25) (layer B.Cu) (net 3))
   (segment (start 242.941234 116.778363) (end 242.340194 116.177323) (width 0.25) (layer B.Cu) (net 4))
-  (segment (start 243.045148 116.882277) (end 242.941234 116.778363) (width 0.25) (layer B.Cu) (net 4))
-  (segment (start 245.003014 116.882277) (end 243.045148 116.882277) (width 0.25) (layer B.Cu) (net 4))
-  (segment (start 245.343188 116.542102) (end 245.003014 116.882277) (width 0.25) (layer B.Cu) (net 4))
-  (segment (start 247.372936 116.542102) (end 245.343188 116.542102) (width 0.25) (layer B.Cu) (net 4))
-  (segment (start 248.050822 117.219988) (end 247.372936 116.542102) (width 0.25) (layer B.Cu) (net 4))
-  (segment (start 248.050822 119.070009) (end 248.050822 117.219988) (width 0.25) (layer B.Cu) (net 4))
-  (segment (start 246.647608 120.473223) (end 248.050822 119.070009) (width 0.25) (layer B.Cu) (net 4))
-  (segment (start 243.431087 107.025413) (end 241.774509 108.681991) (width 0.25) (layer B.Cu) (net 5))
-  (segment (start 244.344163 107.025413) (end 243.431087 107.025413) (width 0.25) (layer B.Cu) (net 5))
+  (segment (start 244.823001 117.406251) (end 243.569122 117.406251) (width 0.25) (layer B.Cu) (net 4))
+  (segment (start 245.68715 116.542102) (end 244.823001 117.406251) (width 0.25) (layer B.Cu) (net 4))
+  (segment (start 243.569122 117.406251) (end 242.941234 116.778363) (width 0.25) (layer B.Cu) (net 4))
+  (segment (start 248.44375 117.612916) (end 247.372936 116.542102) (width 0.25) (layer B.Cu) (net 4))
+  (segment (start 248.44375 118.677081) (end 248.44375 117.612916) (width 0.25) (layer B.Cu) (net 4))
+  (segment (start 247.372936 116.542102) (end 245.68715 116.542102) (width 0.25) (layer B.Cu) (net 4))
+  (segment (start 246.647608 120.473223) (end 248.44375 118.677081) (width 0.25) (layer B.Cu) (net 4))
+  (segment (start 242.693762 108.080951) (end 242.810694 108.197883) (width 0.25) (layer B.Cu) (net 5))
+  (segment (start 241.774509 108.681991) (end 242.375549 108.080951) (width 0.25) (layer B.Cu) (net 5))
+  (segment (start 242.375549 108.080951) (end 242.693762 108.080951) (width 0.25) (layer B.Cu) (net 5))
+  (segment (start 243.171693 108.197883) (end 244.344163 107.025413) (width 0.25) (layer B.Cu) (net 5))
+  (segment (start 242.810694 108.197883) (end 243.171693 108.197883) (width 0.25) (layer B.Cu) (net 5))
   (segment (start 238.83125 87.4125) (end 240.50625 89.0875) (width 0.25) (layer B.Cu) (net 9))
   (segment (start 238.83125 86.075) (end 238.83125 87.4125) (width 0.25) (layer B.Cu) (net 9))

Commit message: OMG ?
Parts:
- removed D3: D_Small, Diode_SMD:D_SOD-123
- added D2: D_Small, Diode_SMD:D_SOD-123, B.Cu at (190.5, 42.1)
- SW1: moved to B.Cu
- moved C2 92.4 mm to (172.1, 63.2), turned to 45 degrees
- moved C1 84.0 mm to (176.9, 74.3), turned to 315 degrees
- moved MX3 73.9 mm to (190.0, 50.0)
- moved C7 73.9 mm to (186.5, 59.5)
- moved C5 73.8 mm to (184.8, 77.5)
- moved C6 73.8 mm to (189.6, 72.8)
- moved Y1 73.8 mm to (187.2, 75.1)
- moved J1 73.7 mm to (180.0, 37.8)
- moved R1 73.7 mm to (178.4, 44.2)
- moved R2 73.7 mm to (180.8, 44.2)
- moved R4 73.7 mm to (173.0, 70.5)
- moved U1 73.7 mm to (180.4, 66.4)
- moved F1 73.7 mm to (183.2, 44.2)
- moved C4 72.9 mm to (176.9, 58.5)
- moved D1 72.3 mm to (170.7, 42.1), turned to 180 degrees
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Connections:
- U1 pad 37: Net-(U1-Pad37) -> ROW0
- U1 pad 38: Net-(U1-Pad38) -> COL1
- U1 pad 39: Net-(U1-Pad39) -> COL0
Routing:
- net +5V: track 0.00 -> 114.2 mm, vias 0 -> 6
- net GND: track 43.8 -> 116.9 mm
- net ROW0: track 0.00 -> 47.5 mm, vias 0 -> 2
- net COL1: track 0.00 -> 24.4 mm, vias 0 -> 2
- net Net-(D1-Pad2): track 0.00 -> 14.1 mm
- net Net-(D2-Pad2): track 0.00 -> 14.0 mm
- net Net-(R3-Pad2): track 0.00 -> 13.4 mm
- net COL0: track 0.00 -> 11.3 mm
- net Net-(C6-Pad1): track 11.0 -> 9.84 mm
- added copper zone on B.Cu, net GND
Other:
- board size 47 x 47 mm -> 45 x 45 mm
