File: Keypad PCB.kicad_pcb (KiCad board)
At the start: 2 copper layers, 45 x 45 mm, 20 parts, among them J1 Conn_01x04_Female, SW1 SW_Push, U1 ATmega32U4-AU, Y1 Crystal_GND24_Small

Commit message: nettoyage
Other:
- net class Default removed
- net class Power removed
