File: Keypad PCB.sch (KiCad schematic (older format))
At the start: 24 parts, among them SW1 SW_Push, U1 ATmega32U4-AU, Y1 Crystal_GND24_Small

Commit message: Avancement sur le rooting du pcb
Parts:
- removed D2, D4: D_Small, Diode_SMD:D_SOD-123, symbol Device:D_Small
- removed MX2, MX4: MX-NoLED, MX_Alps_Hybrid:MX-1U-NoLED, symbol MX_Alps_Hybrid:MX-NoLED
- removed USB1: Molex-0548190589, random-keyboard-parts:Molex-0548190589, symbol random-keyboard-parts:Molex-0548190589
- added J1: Conn_01x04_Female, Connectors_JST:JST_SH_SM04B-SRSS-TB_04x1.00mm_Angled, symbol Connector:Conn_01x04_Female
Connections:
- net GND: now also C5.2, C6.2, J1.1 (Pin_1)
- net VCC: now also J1.4 (Pin_4)
- net D+: no longer names the net of R2.2
- net D+: now also J1.3 (Pin_3)
- net D-: no longer names the net of R1.2
- net D-: now also J1.2 (Pin_2)
Other:
- moved on the sheet: F1
Changed lines of the file:
@@
 Wire Wire Line
 	3450 3100 4900 3100
-Wire Wire Line
-	3950 3000 3000 3000
-Wire Wire Line
-	3250 3100 3000 3100
 $Comp
 L Device:C_Small C7
@@
 Wire Wire Line
 	4700 1500 4700 1550
-Text GLabel 3000 3000 0    50   Input ~ 0
-D+
-Text GLabel 3000 3100 0    50   Input ~ 0
-D-
-$Comp
-L random-keyboard-parts:Molex-0548190589 USB1
-U 1 1 63E36614
-P 8400 2750
-F 0 "USB1" V 8937 2717 60  0000 C CNN
-F 1 "Molex-0548190589" V 8831 2717 60  0000 C CNN
-F 2 "random-keyboard-parts:Molex-0548190589" H 8400 2750 60  0001 C CNN
-F 3 "" H 8400 2750 60  0001 C CNN
-	1    8400 2750
-	0    -1   -1   0
-$EndComp
 $Comp
 L Device:Polyfuse F1
 U 1 1 63E38848
-P 9600 2550
-F 0 "F1" V 9375 2550 50  0000 C CNN
-F 1 "Polyfuse" V 9466 2550 50  0000 C CNN
-F 2 "Fuse:Fuse_1206_3216Metric" H 9650 2350 50  0001 L CNN
-F 3 "~" H 9600 2550 50  0001 C CNN
-	1    9600 2550
+P 2400 2900
+F 0 "F1" V 2175 2900 50  0000 C CNN
+F 1 "Polyfuse" V 2266 2900 50  0000 C CNN
+F 2 "Fuse:Fuse_1206_3216Metric" H 2450 2700 50  0001 L CNN
+F 3 "~" H 2400 2900 50  0001 C CNN
+	1    2400 2900
 	0    1    1    0
 $EndComp
-Wire Wire Line
-	8700 2550 9050 2550
 $Comp
 L power:VCC #PWR0111
 U 1 1 63E3AA5A
-P 9050 2550
-F 0 "#PWR0111" H 9050 2400 50  0001 C CNN
-F 1 "VCC" H 9067 2723 50  0000 C CNN
-F 2 "" H 9050 2550 50  0001 C CNN
-F 3 "" H 9050 2550 50  0001 C CNN
-	1    9050 2550
-	1    0    0    -1
-$EndComp
-Connection ~ 9050 2550
-Wire Wire Line
-	9050 2550 9450 2550
+P 2100 2900
+F 0 "#PWR0111" H 2100 2750 50  0001 C CNN
+F 1 "VCC" H 2117 3073 50  0000 C CNN
+F 2 "" H 2100 2900 50  0001 C CNN
+F 3 "" H 2100 2900 50  0001 C CNN
+	1    2100 2900
+	1    0    0    -1
+$EndComp
 $Comp
 L power:+5V #PWR0112
 U 1 1 63E3BC2B
-P 10000 2550
-F 0 "#PWR0112" H 10000 2400 50  0001 C CNN
-F 1 "+5V" H 10015 2723 50  0000 C CNN
-F 2 "" H 10000 2550 50  0001 C CNN
-F 3 "" H 10000 2550 50  0001 C CNN
-	1    10000 2550
-	1    0    0    -1
-$EndComp
-Wire Wire Line
-	9750 2550 10000 2550
-Text GLabel 8700 2650 2    50   Input ~ 0
-D-
-Text GLabel 8700 2750 2    50   Input ~ 0
-D+
+P 2800 2900
+F 0 "#PWR0112" H 2800 2750 50  0001 C CNN
+F 1 "+5V" H 2815 3073 50  0000 C CNN
+F 2 "" H 2800 2900 50  0001 C CNN
+F 3 "" H 2800 2900 50  0001 C CNN
+	1    2800 2900
+	1    0    0    -1
+$EndComp
 $Comp
 L power:GND #PWR0113
 U 1 1 63E3DCE8
-P 8900 2950
-F 0 "#PWR0113" H 8900 2700 50  0001 C CNN
-F 1 "GND" H 8905 2777 50  0000 C CNN
-F 2 "" H 8900 2950 50  0001 C CNN
-F 3 "" H 8900 2950 50  0001 C CNN
-	1    8900 2950
-	1    0    0    -1
-$EndComp
-Wire Wire Line
-	8700 2950 8900 2950
+P 3000 3200
+F 0 "#PWR0113" H 3000 2950 50  0001 C CNN
+F 1 "GND" H 3005 3027 50  0000 C CNN
+F 2 "" H 3000 3200 50  0001 C CNN
+F 3 "" H 3000 3200 50  0001 C CNN
+	1    3000 3200
+	1    0    0    -1
+$EndComp
 $Comp
 L MX_Alps_Hybrid:MX-NoLED MX1
@@
 	1    0    0    -1
 $EndComp
-$Comp
-L MX_Alps_Hybrid:MX-NoLED MX4
-U 1 1 63E4A8BE
-P 9400 4600
-F 0 "MX4" H 9433 4823 60  0000 C CNN
-F 1 "MX-NoLED" H 9433 4749 20  0000 C CNN
-F 2 "MX_Alps_Hybrid:MX-1U-NoLED" H 8775 4575 60  0001 C CNN
-F 3 "" H 8775 4575 60  0001 C CNN
-	1    9400 4600
-	1    0    0    -1
-$EndComp
-$Comp
-L MX_Alps_Hybrid:MX-NoLED MX2
-U 1 1 63E4B053
-P 8600 4600
-F 0 "MX2" H 8633 4823 60  0000 C CNN
-F 1 "MX-NoLED" H 8633 4749 20  0000 C CNN
-F 2 "MX_Alps_Hybrid:MX-1U-NoLED" H 7975 4575 60  0001 C CNN
-F 3 "" H 7975 4575 60  0001 C CNN
-	1    8600 4600
-	1    0    0    -1
-$EndComp
-$Comp
-L Device:D_Small D2
-U 1 1 63E4C771
-P 8550 5000
-F 0 "D2" V 8596 4932 50  0000 R CNN
-F 1 "D_Small" V 8505 4932 50  0000 R CNN
-F 2 "Diode_SMD:D_SOD-123" V 8550 5000 50  0001 C CNN
-F 3 "~" V 8550 5000 50  0001 C CNN
-	1    8550 5000
-	0    -1   -1   0
-$EndComp
-$Comp
-L Device:D_Small D4
-U 1 1 63E4CE2A
-P 9350 5000
-F 0 "D4" V 9396 4932 50  0000 R CNN
-F 1 "D_Small" V 9305 4932 50  0000 R CNN
-F 2 "Diode_SMD:D_SOD-123" V 9350 5000 50  0001 C CNN
-F 3 "~" V 9350 5000 50  0001 C CNN
-	1    9350 5000
-	0    -1   -1   0
-$EndComp
-Wire Wire Line
-	9350 4750 9350 4900
-Wire Wire Line
-	8550 4750 8550 4900
 $Comp
 L Device:D_Small D1
@@
 $EndComp
 Wire Wire Line
-	8750 3650 8750 4550
-Wire Wire Line
-	9550 3650 9550 4550
-Wire Wire Line
 	8750 3650 8750 3300
-Connection ~ 8750 3650
 Wire Wire Line
 	9550 3650 9550 3300
-Connection ~ 9550 3650
 $Comp
 L Device:D_Small D3
@@
 	8550 4150 8150 4150
 Connection ~ 8550 4150
-Wire Wire Line
-	9350 5100 8550 5100
-Wire Wire Line
-	8550 5100 8150 5100
-Connection ~ 8550 5100
 Text GLabel 8750 3300 1    50   Input ~ 0
 COL0
@@
 Text GLabel 8150 4150 0    50   Input ~ 0
 ROW0
-Text GLabel 8150 5100 0    50   Input ~ 0
-ROW1
+Wire Wire Line
+	3450 2500 3450 2650
+Connection ~ 3450 2500
+Connection ~ 3450 2650
+Wire Wire Line
+	1900 3000 3950 3000
+Wire Wire Line
+	1900 3100 3250 3100
+Wire Wire Line
+	1900 3200 3000 3200
+Wire Wire Line
+	1900 2900 2100 2900
+Wire Wire Line
+	2550 2900 2800 2900
+Connection ~ 2100 2900
+Wire Wire Line
+	2100 2900 2250 2900
+$Comp
+L Connector:Conn_01x04_Female J1
+U 1 1 63ECD72E
+P 1700 3100
+F 0 "J1" H 1592 2675 50  0000 C CNN
+F 1 "Conn_01x04_Female" H 1592 2766 50  0000 C CNN
+F 2 "Connectors_JST:JST_SH_SM04B-SRSS-TB_04x1.00mm_Angled" H 1700 3100 50  0001 C CNN
+F 3 "~" H 1700 3100 50  0001 C CNN
+	1    1700 3100
+	-1   0    0    1
+$EndComp
 $EndSCHEMATC

Commit message: OMG ?
Parts:
- removed D3: D_Small, Diode_SMD:D_SOD-123, symbol Device:D_Small
- added D2: D_Small, Diode_SMD:D_SOD-123, symbol Device:D_Small
Connections:
- net COL0: now also U1.39 (PF4)
- net COL1: now also U1.38 (PF5)
- net ROW0: now also U1.37 (PF6), D2.1 (K)
- net at MX3.2 (ROW): now also D2.2 (A)
Changed lines of the file:
@@
 EESchema Schematic File Version 4
+LIBS:Keypad PCB-cache
 EELAYER 30 0
 EELAYER END
@@
 $EndDescr
 $Comp
-L MCU_Microchip_ATmega:ATmega32U4-AU U1
-U 1 1 63DFA3BE
-P 5500 3500
-F 0 "U1" H 5500 1611 50  0000 C CNN
-F 1 "ATmega32U4-AU" H 5500 1520 50  0000 C CNN
-F 2 "Package_QFP:TQFP-44_10x10mm_P0.8mm" H 5500 3500 50  0001 C CIN
-F 3 "http://ww1.microchip.com/downloads/en/DeviceDoc/Atmel-7766-8-bit-AVR-ATmega16U4-32U4_Datasheet.pdf" H 5500 3500 50  0001 C CNN
-	1    5500 3500
-	1    0    0    -1
-$EndComp
-$Comp
 L power:+5V #PWR0101
 U 1 1 63E012AE
@@
 Wire Wire Line
 	5400 1700 5400 1550
-Wire Wire Line
-	5400 1700 5500 1700
-Connection ~ 5400 1700
-Wire Wire Line
-	5500 1700 5600 1700
-Connection ~ 5500 1700
 $Comp
 L power:GND #PWR0102
@@
 	1    0    0    -1
 $EndComp
-Wire Wire Line
-	4950 5300 5400 5300
-Wire Wire Line
-	5400 5300 5500 5300
-Connection ~ 5400 5300
 $Comp
 L power:GND #PWR0103
@@
 $EndComp
 Wire Wire Line
-	6100 4100 6700 4100
-Wire Wire Line
 	6900 4100 7500 4100
 $Comp
@@
 	1    0    0    -1
 $EndComp
-Wire Wire Line
-	8550 3850 8550 3950
 $Comp
 L MX_Alps_Hybrid:MX-NoLED MX3
@@
 	1    0    0    -1
 $EndComp
-$Comp
-L Device:D_Small D1
-U 1 1 63E40E4C
-P 8550 4050
-F 0 "D1" V 8596 3982 50  0000 R CNN
-F 1 "D_Small" V 8505 3982 50  0000 R CNN
-F 2 "Diode_SMD:D_SOD-123" V 8550 4050 50  0001 C CNN
-F 3 "~" V 8550 4050 50  0001 C CNN
-	1    8550 4050
-	0    -1   -1   0
-$EndComp
 Wire Wire Line
 	8750 3650 8750 3300
 Wire Wire Line
 	9550 3650 9550 3300
-$Comp
-L Device:D_Small D3
-U 1 1 63E57EF8
-P 9350 4050
-F 0 "D3" V 9396 3982 50  0000 R CNN
-F 1 "D_Small" V 9305 3982 50  0000 R CNN
-F 2 "Diode_SMD:D_SOD-123" V 9350 4050 50  0001 C CNN
-F 3 "~" V 9350 4050 50  0001 C CNN
-	1    9350 4050
-	0    -1   -1   0
-$EndComp
-Wire Wire Line
-	9350 3850 9350 3950
-Wire Wire Line
-	9350 4150 8550 4150
-Wire Wire Line
-	8550 4150 8150 4150
-Connection ~ 8550 4150
 Text GLabel 8750 3300 1    50   Input ~ 0
 COL0
 Text GLabel 9550 3300 1    50   Input ~ 0
 COL1
-Text GLabel 8150 4150 0    50   Input ~ 0
-ROW0
 Wire Wire Line
 	3450 2500 3450 2650
@@
 	-1   0    0    1
 $EndComp
+Connection ~ 5400 5300
+Wire Wire Line
+	4950 5300 5400 5300
+Connection ~ 5500 1700
+Connection ~ 5400 1700
+Wire Wire Line
+	6100 4100 6700 4100
+Wire Wire Line
+	5500 1700 5600 1700
+Wire Wire Line
+	5400 5300 5500 5300
+Wire Wire Line
+	5400 1700 5500 1700
+Text GLabel 6200 4700 2    50   Input ~ 0
+COL1
+Text GLabel 6200 4600 2    50   Input ~ 0
+COL0
+$Comp
+L MCU_Microchip_ATmega:ATmega32U4-AU U1
+U 1 1 63DFA3BE
+P 5500 3500
+F 0 "U1" H 5500 1611 50  0000 C CNN
+F 1 "ATmega32U4-AU" H 5500 1520 50  0000 C CNN
+F 2 "Package_QFP:TQFP-44_10x10mm_P0.8mm" H 5500 3500 50  0001 C CIN
+F 3 "http://ww1.microchip.com/downloads/en/DeviceDoc/Atmel-7766-8-bit-AVR-ATmega16U4-32U4_Datasheet.pdf" H 5500 3500 50  0001 C CNN
+	1    5500 3500
+	1    0    0    -1
+$EndComp
+Wire Wire Line
+	6100 4600 6200 4600
+Wire Wire Line
+	6100 4700 6200 4700
+$Comp
+L Device:D_Small D1
+U 1 1 63E15488
+P 8450 3950
+F 0 "D1" V 8496 3882 50  0000 R CNN
+F 1 "D_Small" V 8405 3882 50  0000 R CNN
+F 2 "Diode_SMD:D_SOD-123" V 8450 3950 50  0001 C CNN
+F 3 "~" V 8450 3950 50  0001 C CNN
+	1    8450 3950
+	0    -1   -1   0
+$EndComp
+$Comp
+L Device:D_Small D2
+U 1 1 63E15EE0
+P 9250 3950
+F 0 "D2" V 9296 3882 50  0000 R CNN
+F 1 "D_Small" V 9205 3882 50  0000 R CNN
+F 2 "Diode_SMD:D_SOD-123" V 9250 3950 50  0001 C CNN
+F 3 "~" V 9250 3950 50  0001 C CNN
+	1    9250 3950
+	0    -1   -1   0
+$EndComp
+Wire Wire Line
+	8450 3850 8550 3850
+Wire Wire Line
+	9250 3850 9350 3850
+Wire Wire Line
+	8250 4050 8450 4050
+Connection ~ 8450 4050
+Wire Wire Line
+	8450 4050 9250 4050
+Text GLabel 8250 4050 0    50   Input ~ 0
+ROW0
+Text GLabel 6100 4800 2    50   Input ~ 0
+ROW0
 $EndSCHEMATC
